File: Hardware_design/KICAD_project/fly_control_board/fly_control_board.sch (KiCad schematic (older format))
At the start: 1 part

Commit message: Nick_Zheng Start Drawing Board
先仿着参考原理图自己画了一下，当作是学习
Parts:
- added C1, C2, C3, C5: 12pF, symbol Device:C_Small
- added C10, C11, C12, C9: 100nF, Capacitor_SMD:C_0603_1608Metric, symbol Device:C_Small
- added C13, C14: 10uF, symbol Device:C_Small
- added C4, C8: 100nF, symbol Device:C_Small
- added C6: 22uF, Capacitor_SMD:C_0603_1608Metric, symbol Device:C_Small
- added C7: 10uF, Capacitor_SMD:C_0603_1608Metric, symbol Device:C_Small
- added D1, D4: CESD3V3D3, symbol Device:D
- added D2: LED3_0603_1608Metric, LED_SMD:LED_0603_1608Metric, symbol Device:LED
- added D3: LED2_0603_1608Metric, LED_SMD:LED_0603_1608Metric, symbol Device:LED
- added J?: USB_C_Receptacle_USB2.0, Connector_USB:USB_C_Receptacle_Palconn_UTC16-G, symbol Connector:USB_C_Receptacle_USB2.0
- added J?: Micro_SD_Card, symbol Connector:Micro_SD_Card
- added R1, R3: 10K, symbol Device:R_Small
- added R14, R15, R2, R6, R7: 10K, Resistor_SMD:R_0603_1608Metric, symbol Device:R_Small
- added R4, R9: 4.7K, Resistor_SMD:R_0603_1608Metric, symbol Device:R_Small
- added SW1: SW_Normally_Open, Button_Switch_SMD:SW_Push_1P1T_NO_6x6mm_H9.5mm, symbol Switch:SW_Push
- added U1: AMS1117-3.3, Package_TO_SOT_SMD:SOT-223-3_TabPin2, symbol Regulator_Linear:AMS1117-3.3
- added U2: LY68L6400SLIT, Package_SO:SOIC-8_3.9x4.9mm_P1.27mm, symbol Memory_Flash:W25Q32JVSS
- added U4: W25Q64JVSS, Package_SO:SOIC-8_5.23x5.23mm_P1.27mm, symbol Memory_Flash:W25Q32JVSS
- added U5: W25Q32JVSS, Package_SO:SOIC-8_5.23x5.23mm_P1.27mm, symbol Memory_Flash:W25Q32JVSS
- added X1: 32.768kHz, symbol Device:Crystal
- added X2: 32MHz, symbol Device:Crystal_GND24_Small
- gave numbers to parts that had none: 1
Connections:
- net SQPI_IO2: now reaches U3.1 (PE2)
- net GND: now reaches U3.10 (VSS)
- net GND: now also U3.19 (VSSA), U3.26 (VSS), U3.49 (VSS), U3.74 (VSS), U3.99 (VSS), C1.1, C10.2, C11.2, C12.2, C13.2, C14.2, C2.1, C3.2, C4.1, C5.1, C6.2, C7.2, C8.2, C9.2, J?.6 (VSS), J?.9 (SHIELD), J?.A1 (GND), J?.A12 (GND), J?.B1 (GND), J?.B12 (GND), J?.S1 (SHIELD), R14.2, R15.2, R3.2, R4.2, R9.2, SW1.2, U1.1 (GND), U2.4 (GND), U4.4 (GND), U5.4 (GND), X2.2, X2.4
- net 3V3: now reaches U3.100 (VDD)
- net 3V3: now also U3.11 (VDD), U3.20 (VREF+), U3.21 (VDDA), U3.27 (VDD), U3.50 (VDD), U3.6 (VBAT), U3.75 (VDD), C10.1, C11.1, C12.1, C7.1, C8.1, C9.1, D1.2 (A), J?.4 (VDD), R1.1, R2.1, R6.1, R7.1, U1.2 (VO), U2.8 (VCC), U4.8 (VCC), U5.8 (VCC)
- net OSCIN: now reaches U3.12 (PH0)
- net OSCIN: now also C3.1, X2.1
- net OSCOUT: now reaches U3.13 (PH1)
- net OSCOUT: now also C5.2, X2.3
- net NRST: now reaches U3.14 (NRST)
- net NRST: now also C4.2, R1.2, SW1.1
- net MEM_FLASHCS: now reaches U3.15 (PC0)
- net MEM_FLASHCS: now also R7.2, U5.1 (~CS)
- net MEM_MISO: now reaches U3.17 (PC2_C)
- net MEM_MISO: now also U2.2 (DO(IO1)), U5.2 (DO(IO1))
- net MEM_MOSI: now reaches U3.18 (PC3_C)
- net MEM_MOSI: now also U2.5 (DI(IO0)), U5.5 (DI(IO0))
- net SD_CMD: now reaches U3.22 (PA0)
- net SD_CMD: now also J?.3 (CMD)
- net QSPI_SCK: now reaches U3.36 (PB2)
- net QSPI_SCK: now also U4.6 (CLK)
- net LEDR: now reaches U3.4 (PE5)
- net LEDR: now also D2.2 (A)
- net MEM_SCK: now reaches U3.46 (PB10)
- net MEM_SCK: now also U2.6 (CLK), U5.6 (CLK)
- net at U3.48 (VCAP1): now also C13.1
- net LEDG: now reaches U3.5 (PE6)
- net LEDG: now also D3.2 (A)
- net SD_D0: now reaches U3.53 (PB14)
- net SD_D0: now also J?.7 (DAT0)
- net SD_D1: now reaches U3.54 (PB15)
- net SD_D1: now also J?.8 (DAT1)
- net QSPI_IO3: now reaches U3.60 (PD13)
- net QSPI_IO3: now also U4.7 (IO3)
- net QSPI_IO0: now reaches U3.66 (PC9)
- net QSPI_IO0: now also U4.5 (DI(IO0))
- net MEM_PSRAMCS: now reaches U3.7 (PC13)
- net MEM_PSRAMCS: now also R2.2, U2.1 (~CS)
- net USB_N: now reaches U3.70 (PA11)
- net USB_N: now also J?.A7 (D-), J?.B7 (D-)
- net USB_P: now reaches U3.71 (PA12)
- net USB_P: now also J?.A6 (D+), J?.B6 (D+)
- net TMS: now reaches U3.72 (PA13)
- net at U3.73 (VCAP2): now also C14.1
- net TCK: now reaches U3.76 (PA14)
- net QSPI_IO1: now reaches U3.78 (PC10)
- net QSPI_IO1: now also U4.2 (DO(IO1))
- net OSC32IN: now reaches U3.8 (PC14)
- net OSC32IN: now also C1.2, X1.1
- net SD_CLK: now reaches U3.87 (PD6)
- net SD_CLK: now also J?.5 (CLK)
- net SD_D2: now reaches U3.89 (PB3)
- net SD_D2: now also J?.1 (DAT2)
- net OSC32OUT: now reaches U3.9 (PC15)
- net OSC32OUT: now also C2.2, X1.2
- net SD_D3: now reaches U3.90 (PB4)
- net SD_D3: now also J?.2 (DAT3/CD)
- net QSPI_CS: now reaches U3.92 (PB6)
- net QSPI_CS: now also R6.2, U4.1 (~CS)
- net BOOT0: now reaches U3.94 (BOOT0)
- net BOOT0: now also R3.1
- new net: D2.1 (K), R15.1
- new net: D3.1 (K), R14.1
- new net: J?.A5 (CC1), R9.1
- new net: J?.B5 (CC2), R4.1
- new net QSPI_IO2: U4.3 (IO2)
- new net VBAT: D4.2 (A)
- new net VBUS: C6.1, J?.A4 (VBUS), J?.A9 (VBUS), J?.B4 (VBUS), J?.B9 (VBUS), U1.3 (VI)
- new net _VBAT: D1.1 (K), D4.1 (K)
- no-connect marks 0 -> 6
Other:
- note added: "MEM"
- note added: "Main_Clock_Crystal\n"
- note added: "RTC_Clock_Crystal"
- moved on the sheet: U3
