File: Hardware_design/KICAD_project/upper_board/upper_board.kicad_pcb (KiCad board)
At the start: 2 copper layers, 137 parts, among them J1 USBC_16P_4MP-connector, J2 Conn_02x05_Counter_Clockwise, J3 Conn_02x07_Counter_Clockwise, J4 Conn_02x08_Counter_Clockwise, J5 Conn_01x04, J6 Conn_01x02_Female, J7 Conn_02x03_Counter_Clockwise, SW1 SW_Push, U1 CH340C, U2 mcu_STM32H750VBT6, U3 AP1117-33, U4 W25Q128JVS, U5 ICM-20602, U6 BMI160, U7 IST8310, Y1 32.768kHz, Y2 32MHz

Commit message: 控制系统硬件设计完成，电源板正式发布v1.0.0 控制板打样v0.2.0测试
Parts:
- removed J5: Conn_01x04, upper_board:OLED_0.96
- removed J7: Conn_02x03_Counter_Clockwise, Connector_PinHeader_1.27mm:PinHeader_2x03_P1.27mm_Horizontal
- removed R11, R21, R25, R48, R49: 22, Resistor_SMD:R_0603_1608Metric_Pad0.98x0.95mm_HandSolder
- removed R58: 4.7k, Resistor_SMD:R_0603_1608Metric_Pad0.98x0.95mm_HandSolder
- removed R60, R61, R62, R63: 10K, Resistor_SMD:R_0603_1608Metric_Pad0.98x0.95mm_HandSolder
- removed R72, R73, R74, R75, R76, R77: 0, Resistor_SMD:R_0603_1608Metric_Pad0.98x0.95mm_HandSolder
- added C27: 100nF, Capacitor_SMD:C_0603_1608Metric_Pad1.08x0.95mm_HandSolder, F.Cu at (120.0, 92.8)
- added C28: 100nF, Capacitor_SMD:C_0603_1608Metric_Pad1.08x0.95mm_HandSolder, B.Cu at (124.5, 93.5)
- added C29: 0.1uF, Capacitor_SMD:C_0603_1608Metric_Pad1.08x0.95mm_HandSolder, F.Cu at (120.0, 94.5)
- added C30: 0.1uF, Capacitor_SMD:C_0603_1608Metric_Pad1.08x0.95mm_HandSolder, B.Cu at (121.4, 97.5)
- added G***: LOGO, batt_board:small_404APD, F.Cu at (122.7, 72.1)
- added U8: BMP280, Package_LGA:Bosch_LGA-8_2x2.5mm_P0.65mm_ClockwisePinNumbering, F.Cu at (123.3, 92.6)
- C1, C12, C18, C2, C3, C4, C5, C7, C8, J4, R18, R22, R23, R26, R27, R28, R29, R30, R31, R32, R33, R34, R35, R4, R43, R44, R45, R46, R47, R5, R52, R53, R56, R57, R6, R65, R67, R68, R69, R7, U3: moved to B.Cu
- C9: value 100nF/0.1uF -> 100nF; moved to B.Cu
- J2: value Conn_02x05_Counter_Clockwise -> Conn_02x03_Counter_Clockwise; footprint Connector_PinSocket_2.54mm:PinSocket_2x05_P2.54mm_Horizontal -> Connector_PinHeader_1.27mm:PinHeader_2x03_P1.27mm_Vertical_SMD; moved to B.Cu
- J3: footprint Connector_PinHeader_1.00mm:PinHeader_2x07_P1.00mm_Horizontal -> Connector_PinHeader_2.54mm:PinHeader_2x07_P2.54mm_Vertical_SMD; moved to B.Cu
- J6: value Conn_01x02_Female -> Conn_01x03; footprint Button_Switch_SMD:ESC_Battery_Pale -> Connector_PinHeader_2.54mm:PinHeader_1x03_P2.54mm_Vertical
- moved R36 276.4 mm to (127.1, 86.1)
- moved R33 273.2 mm to (130.2, 83.8)
- moved R32 271.7 mm to (128.2, 104.3), turned to 90 degrees
- moved R19 270.9 mm to (119.3, 84.6)
- moved C10 270.5 mm to (131.0, 92.7), turned to 270 degrees
- moved R67 269.8 mm to (127.3, 92.3)
- moved R15 268.4 mm to (130.7, 76.6)
- moved R14 268.4 mm to (130.7, 75.1)
- moved R54 267.9 mm to (135.9, 97.8), turned to 90 degrees
- moved R38 267.3 mm to (127.2, 89.3)
- moved R44 266.1 mm to (133.5, 65.8), turned to 270 degrees
- moved R10 264.8 mm to (136.9, 74.4), turned to 270 degrees
- moved R66 262.8 mm to (141.4, 66.0), turned to 90 degrees
- moved C25 262.6 mm to (132.2, 68.4)
- moved R71 261.2 mm to (125.5, 99.4)
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Connections:
- C12 pad 1: /VBUS -> +5V
- C7 pad 2: /VBUS -> +5V
- C8 pad 2: /VBUS -> +5V
- D9 pad 1: GND -> Net-(D9-Pad1)
- J1 pad A4: /VBUS -> +5V
- J1 pad A9: /VBUS -> +5V
- J1 pad B4: /VBUS -> +5V
- J1 pad B9: /VBUS -> +5V
- J2 pad 1: +3V3 -> /TIM1_CH1
- J2 pad 2: Net-(J2-Pad2) -> /TIM1_CH2
- J2 pad 3: +5V -> /TIM1_CH3
- J2 pad 4: Net-(J2-Pad4) -> /TIM1_CH4
- J2 pad 5: /TIM3_CH3 -> /ADC2_INP3
- J2 pad 6: /TIM1_CH4 -> /TIM3_CH3
- J3 pad 10: /TIM2_CH2 -> /TIM2_CH3
- J3 pad 11: /TIM2_CH1 -> /TIM2_CH4
- J3 pad 8: /TIM2_CH4 -> /TIM2_CH1
- J3 pad 9: /TIM2_CH3 -> /TIM2_CH2
- J6 pad 1: GND -> +3V3
- J6 pad 2: Net-(J6-Pad2) -> GND
- R32 pad 1: /UART4_TX_RX -> Net-(D9-Pad1)
- R32 pad 2: +3V3 -> GND
- U1 pad 16: /VBUS -> +5V
- U3 pad 3: /VBUS -> +5V
- U7 pad 13: Net-(R72-Pad1) -> +3V3
- U7 pad 2: Net-(R73-Pad1) -> +3V3
- U7 pad 5: Net-(R74-Pad2) -> GND
- U7 pad 6: Net-(R75-Pad1) -> GND
Routing:
- net +3V3: track 0.00 -> 344.6 mm, vias 0 -> 28
- net GND: track 0.00 -> 199.2 mm, vias 0 -> 49
- net +5V: track 0.00 -> 102.1 mm, vias 0 -> 4
- net /QSPI_CLK: track 0.00 -> 49.6 mm, vias 0 -> 7
- net /QSPI_IO3: track 0.00 -> 41.1 mm, vias 0 -> 4
- net Net-(R43-Pad2): track 0.00 -> 38.6 mm, vias 0 -> 1
- net /TIM2_CH2: track 0.00 -> 38.1 mm, vias 0 -> 4
- net Net-(R44-Pad2): track 0.00 -> 36.2 mm, vias 0 -> 2
- net /QSPI_~CS: track 0.00 -> 33.2 mm, vias 0 -> 2
- net /I2C1_SDA: track 0.00 -> 32.9 mm
- net /SCK: track 0.00 -> 32.6 mm, vias 0 -> 5
- net /SPI1_MISO: track 0.00 -> 30.1 mm
- net /NRST: track 0.00 -> 29.3 mm, vias 0 -> 2
- net /BMI_~CS: track 0.00 -> 28.8 mm, vias 0 -> 3
- net /I2C1_SCL: track 0.00 -> 26.0 mm, vias 0 -> 4
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- added copper zone on B.Cu, net GND
- added copper zone on F.Cu, net GND
Other:
- board outline added: 50 x 50 mm
- board text added: "3.3v GND TIM2_CH3 TIM2_CH1 SPI1_MISO I2C1_SCL UART7_RX_TX"
- board text added: "5v TIM2_CH4 TIM2_CH2 SPI1_SCK SPI1_MOSI I2C1_SDA UART7_TX_RX"
