File: Hardware_design/KICAD_project/upper_board/upper_board.sch (KiCad schematic (older format))
At the start: 92 parts

Commit message: 完善了供电板，增加了 IMU的外围传感电路设计
Parts:
- removed J?: Micro_SD_Card_Det, Connector_Card:microSD_HC_Hirose_DM3D-SF, symbol Connector:Micro_SD_Card_Det
- added C? (x2): 0.1uF, symbol Device:C_Small
- added C?: 2.2uF, symbol Device:C_Small
- added C? (x7): C_Small, symbol Device:C_Small
- added R?: R_Small, symbol Device:R_Small
Connections:
- net labels added: 3.3V, BMI_~CS, DRDY, ICM_~CS, ISTRES_PIN, ITS_~RST, SCK, SD0, SD1, SDA_I2C, SDI
- wire segments 147 -> 239
- no-connect marks 5 -> 15
Other:
- moved on the sheet: C?, D?, J?, R?, U?

Commit message: upper board design is  completed
Parts:
- removed C? (x29): C_Small, symbol Device:C_Small
- removed D? (x15): LED_Small, symbol Device:LED_Small
- removed J?: Conn_02x08_Counter_Clockwise, symbol Connector_Generic:Conn_02x08_Counter_Clockwise
- removed J?: Conn_01x07_Male, symbol Connector:Conn_01x07_Male
- removed J?: Conn_ARM_JTAG_SWD_20, symbol Connector:Conn_ARM_JTAG_SWD_20
- removed J?: Conn_02x12_Counter_Clockwise, symbol Connector_Generic:Conn_02x12_Counter_Clockwise
- removed R? (x20): R_Small, symbol Device:R_Small
- added C10, C11, C7: 10uF, Capacitor_SMD:C_0603_1608Metric_Pad1.08x0.95mm_HandSolder, symbol Device:C_Small
- added C18, C19, C6: 100nF, Capacitor_SMD:C_0603_1608Metric_Pad1.08x0.95mm_HandSolder, symbol Device:C_Small
- added C23: 10nF, Capacitor_SMD:C_0603_1608Metric_Pad1.08x0.95mm_HandSolder, symbol Device:C_Small
- added C8: 0.1uF, Capacitor_SMD:C_0603_1608Metric_Pad1.08x0.95mm_HandSolder, symbol Device:C_Small
- added C9: 100nF/0.1uF, Capacitor_SMD:C_0603_1608Metric_Pad1.08x0.95mm_HandSolder, symbol Device:C_Small
- added D1, D10, D11, D12, D2, D3, D4, D7, D8, D9: LED_Small, LED_SMD:LED_0603_1608Metric_Pad1.05x0.95mm_HandSolder, symbol Device:LED_Small
- added H1, H2, H3, H4: MountingHole_Pad, MountingHole:MountingHole_3.2mm_M3_DIN965_Pad, symbol Mechanical:MountingHole_Pad
- added J3: Conn_02x07_Counter_Clockwise, Connector_PinHeader_1.00mm:PinHeader_2x07_P1.00mm_Horizontal, symbol Connector_Generic:Conn_02x07_Counter_Clockwise
- added J4: Conn_02x08_Counter_Clockwise, upper_board:BLT_foot print, symbol Connector_Generic:Conn_02x08_Counter_Clockwise
- added J5: Conn_01x04, upper_board:OLED_0.96, symbol Connector_Generic:Conn_01x04
- added J6: Conn_01x02_Female, Button_Switch_SMD:ESC_Battery_Pale, symbol Connector:Conn_01x02_Female
- added J7: Conn_02x03_Counter_Clockwise, Connector_PinHeader_1.27mm:PinHeader_2x03_P1.27mm_Horizontal, symbol Connector_Generic:Conn_02x03_Counter_Clockwise
- added R10, R11, R12, R13, R14, R15, R16, R17, R18, R19, R21, R22, R23, R24, R25, R27, R28, R29, R30, R33, R34, R35, R36, R37, R38, R39, R40, R41, R42, R43, R44, R45, R46, R47, R48, R49, R50, R51, R52, R53, R54, R55, R8, R9: 22, Resistor_SMD:R_0603_1608Metric_Pad0.98x0.95mm_HandSolder, symbol Device:R_Small
- added R26, R31, R32, R4, R5, R56, R57, R58, R6, R65, R67, R68, R7, R71: 4.7k, Resistor_SMD:R_0603_1608Metric_Pad0.98x0.95mm_HandSolder, symbol Device:R_Small
- added R59, R66, R70: 10k, Resistor_SMD:R_0603_1608Metric_Pad0.98x0.95mm_HandSolder, symbol Device:R_Small
- added R60, R61, R62, R63, R69: 10K, Resistor_SMD:R_0603_1608Metric_Pad0.98x0.95mm_HandSolder, symbol Device:R_Small
- added R72, R73, R74, R75, R76, R77: 0, Resistor_SMD:R_0603_1608Metric_Pad0.98x0.95mm_HandSolder, symbol Device:R_Small
- added SW1: SW_Push, upper_board:push_botton, symbol Switch:SW_Push
- added SWD1: Conn_01x05_Male, Connector_PinSocket_2.54mm:PinSocket_1x05_P2.54mm_Vertical, symbol Connector:Conn_01x05_Male
- added U3: AP1117-33, Package_TO_SOT_SMD:SOT-223-3_TabPin2, symbol Regulator_Linear:AP1117-33
- C1, C2, C20, C21, C25: renamed from C?; footprint (none) -> Capacitor_SMD:C_0603_1608Metric_Pad1.08x0.95mm_HandSolder
- C12: renamed from C?; value C_Small -> 22uF; footprint (none) -> Capacitor_SMD:C_0603_1608Metric_Pad1.08x0.95mm_HandSolder
- C13: renamed from C?; value C_Small -> 10uF; footprint (none) -> Capacitor_SMD:C_0603_1608Metric_Pad1.08x0.95mm_HandSolder
- C14, C15, C16, C17, C22, C24, C5: renamed from C?; value C_Small -> 100nF; footprint (none) -> Capacitor_SMD:C_0603_1608Metric_Pad1.08x0.95mm_HandSolder
- C26: renamed from C?; value C_Small -> 4.7uF; footprint (none) -> Capacitor_SMD:C_0603_1608Metric_Pad1.08x0.95mm_HandSolder
- C3, C4: renamed from C?; value C_Small -> 12pF; footprint (none) -> Capacitor_SMD:C_0603_1608Metric_Pad1.08x0.95mm_HandSolder
- D5, D6: renamed from D?; footprint (none) -> LED_SMD:LED_0603_1608Metric_Pad1.05x0.95mm_HandSolder
- J2: renamed from J?; footprint (none) -> Connector_PinSocket_2.54mm:PinSocket_2x05_P2.54mm_Horizontal
- R1, R2: renamed from R?; value R_Small -> 4.7k; footprint (none) -> Resistor_SMD:R_0603_1608Metric_Pad0.98x0.95mm_HandSolder
- R20, R64: renamed from R?; value R_Small -> 10k; footprint (none) -> Resistor_SMD:R_0603_1608Metric_Pad0.98x0.95mm_HandSolder
- R3: renamed from R?; value R_Small -> 10K; footprint (none) -> Resistor_SMD:R_0603_1608Metric_Pad0.98x0.95mm_HandSolder
- U2: renamed from U?; footprint LQFP-100_14x14mm_P0.5mm -> Package_QFP:LQFP-100_14x14mm_P0.5mm
- Y1: renamed from Y?; footprint (none) -> upper_board:LSE_3215
- Y2: renamed from Y?; value Crystal_GND24 -> 32MHz; footprint (none) -> Oscillator:Oscillator_SMD_Abracon_ASE-4Pin_3.2x2.5mm_HandSoldering
- gave numbers to parts that had none: 6
Connections:
- net labels added: ADC2_INP3, ADC2_INP4, ADC3_INP1, BLT_RST, I2C1_SCL, I2C1_SDA, I2C2_SCL, I2C2_SDA, NRST, QSPI_CLK, QSPI_IO0, QSPI_IO1, QSPI_IO3, QSPI_~CS, SPI1_MISO, SPI1_MOSI, SPI1_SCK, SPI2_MISO, SPI2_MOSI, SPI2_SCK, SWDCLK, SWDIO, TIM1_CH1, TIM1_CH2, TIM1_CH3, TIM1_CH4, TIM2_CH1, TIM2_CH2, TIM2_CH3, TIM2_CH4, TIM3_CH1, TIM3_CH2, TIM3_CH3, TIM3_CH4, UART4_RX_TX, UART4_TX_RX, UART5_RX_TX, UART5_TX_RX, UART7_RX_TX, UART7_TX_RX, USB_N, USB_P
- net labels removed: 3.3V, ISTRES_PIN, PPM, PWM_CH1, PWM_CH2, PWM_CH3, PWM_CH4, RXD, SD1, SDA_I2C, SD_CDN, TXD, _VBAT
- wire segments 239 -> 342
- no-connect marks 15 -> 60
Other:
- note added: "1117\n"
- note added: "ADC\n"
- note added: "Mount Hole\n"
- note added: "RX need 3.3V and 10K risister to pull up\n"
- note added: "check 2021.2.27\n"
- note added: "extend\n"
- note removed: "TF set\n"
- moved on the sheet: C1, C12, C13, C14, C15, C16, C17, C2, C20, C21, C22, C24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

Commit message: 控制系统硬件设计完成，电源板正式发布v1.0.0 控制板打样v0.2.0测试
Parts:
- removed J2: Conn_02x05_Counter_Clockwise, Connector_PinSocket_2.54mm:PinSocket_2x05_P2.54mm_Horizontal, symbol Connector_Generic:Conn_02x05_Counter_Clockwise
- removed J5: Conn_01x04, upper_board:OLED_0.96, symbol Connector_Generic:Conn_01x04
- removed J6: Conn_01x02_Female, Button_Switch_SMD:ESC_Battery_Pale, symbol Connector:Conn_01x02_Female
- removed J7: Conn_02x03_Counter_Clockwise, Connector_PinHeader_1.27mm:PinHeader_2x03_P1.27mm_Horizontal, symbol Connector_Generic:Conn_02x03_Counter_Clockwise
- removed R11, R21, R25, R48, R49: 22, Resistor_SMD:R_0603_1608Metric_Pad0.98x0.95mm_HandSolder, symbol Device:R_Small
- removed R58: 4.7k, Resistor_SMD:R_0603_1608Metric_Pad0.98x0.95mm_HandSolder, symbol Device:R_Small
- removed R60, R61, R62, R63: 10K, Resistor_SMD:R_0603_1608Metric_Pad0.98x0.95mm_HandSolder, symbol Device:R_Small
- removed R72, R73, R74, R75, R76, R77: 0, Resistor_SMD:R_0603_1608Metric_Pad0.98x0.95mm_HandSolder, symbol Device:R_Small
- added C27, C28: 100nF, Capacitor_SMD:C_0603_1608Metric_Pad1.08x0.95mm_HandSolder, symbol Device:C_Small
- added C29, C30: 0.1uF, Capacitor_SMD:C_0603_1608Metric_Pad1.08x0.95mm_HandSolder, symbol Device:C_Small
- added J2: Conn_02x03_Counter_Clockwise, Connector_PinHeader_1.27mm:PinHeader_2x03_P1.27mm_Vertical_SMD, symbol Connector_Generic:Conn_02x03_Counter_Clockwise
- added J6: Conn_01x03, Connector_PinHeader_2.54mm:PinHeader_1x03_P2.54mm_Vertical, symbol Connector_Generic:Conn_01x03
- added U8: BMP280, Package_LGA:Bosch_LGA-8_2x2.5mm_P0.65mm_ClockwisePinNumbering, symbol Sensor_Pressure:BMP280
- C9: value 100nF/0.1uF -> 100nF
- J3: footprint Connector_PinHeader_1.00mm:PinHeader_2x07_P1.00mm_Horizontal -> Connector_PinHeader_2.54mm:PinHeader_2x07_P2.54mm_Vertical_SMD
Connections:
- net VBUS is gone; now on net +5V: C12.1, C7.2, C8.2, J1.A4 (VBUS), J1.A9 (VBUS), J1.B4 (VBUS), J1.B9 (VBUS), U1.16 (VCC), U3.3 (VI)
- net +3V3: now also U7.13 (DVDD), U7.2 (AVDD), C27.1, C28.2, C29.1, C30.2, J6.1 (Pin_1), U8.2 (CSB), U8.6 (VDDIO), U8.8 (VDD); no longer R32.2
- net +5V: now also J6.3 (Pin_3)
- net ADC2_INP3: now also J2.5 (Pin_5)
- net GND: now also R32.2, U7.5 (CAD0), U7.6 (CAD1), C27.2, C28.1, C29.2, C30.1, J6.2 (Pin_2), U8.1 (GND), U8.5 (SDO), U8.7 (GND); no longer D9.1 (K)
- net I2C2_SCL: now also U8.4 (SCK)
- net I2C2_SDA: now also U8.3 (SDI)
- net TIM1_CH1: now also J2.1 (Pin_1)
- net TIM1_CH2: now also J2.2 (Pin_2)
- net TIM1_CH3: now also J2.3 (Pin_3)
- net TIM1_CH4: now also J2.4 (Pin_4)
- net TIM2_CH1: now also J3.8 (Pin_8); no longer J3.11 (Pin_11)
- net TIM2_CH2: now also J3.9 (Pin_9); no longer J3.10 (Pin_10)
- net TIM2_CH3: now also J3.10 (Pin_10); no longer J3.9 (Pin_9)
- net TIM2_CH4: now also J3.11 (Pin_11); no longer J3.8 (Pin_8)
- net TIM3_CH3: now also J2.6 (Pin_6)
- net UART4_TX_RX: no longer R32.1
- new net: D9.1 (K), R32.1
- no-connect marks 60 -> 62
Other:
- note added: "TIM2 can be used as chip choose signal\n"
- note removed: "ADC\n"
- moved on the sheet: C1, C10, C11, C2, C3, C4, C5, C6, D1, D2, D3, D4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
